File: task/task-v/eagle/task-43/ground_truth/answer.sch (EAGLE design)
At the start: 0 parts

Commit message: Refine engineering task metadata and instructions
Changed lines of the file:
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@@
 </classes>
 <parts>
-<part name="U1" library="linear" deviceset="*555" device="N"/>
+<part name="U1" library="linear" deviceset="LM358" device=""/>
+<part name="R1" library="rcl" deviceset="R-EU_" device="0207/10" value="10k"/>
+<part name="C1" library="rcl" deviceset="C-EU" device="025-025X050" value="100n"/>
+<part name="U1_1" library="linear" deviceset="LM358" device=""/>
+<part name="R1_1" library="rcl" deviceset="R-EU_" device="0207/10" value="10k"/>
+<part name="C1_1" library="rcl" deviceset="C-EU" device="025-025X050" value="100n"/>
 </parts>
 <sheets>
@@
 <plain></plain>
 <instances>
-<instance part="U1" gate="A" x="50" y="40"/>
+<instance part="U1" gate="A" x="50.8" y="50.8"/>
+<instance part="R1" gate="G$1" x="40.64" y="45.72" rot="R90"/>
+<instance part="C1" gate="G$1" x="60.96" y="45.72"/>
+<instance part="U1_1" gate="A" x="101.6" y="50.8"/>
+<instance part="R1_1" gate="G$1" x="91.44" y="45.72" rot="R90"/>
+<instance part="C1_1" gate="G$1" x="111.76" y="45.72"/>
 </instances>
 <busses></busses>
 <nets>
+<net name="IN" class="0">
+<segment>
+<pinref part="U1" gate="A" pin="IN+"/>
+<pinref part="R1" gate="G$1" pin="1"/>
+<wire x1="40.64" y1="45.72" x2="50.8" y2="45.72" width="0.1524" layer="91"/>
+</segment>
+</net>
+<net name="OUT" class="0">
+<segment>
+<pinref part="U1" gate="A" pin="OUT"/>
+<pinref part="C1" gate="G$1" pin="1"/>
+<wire x1="55.88" y1="50.8" x2="60.96" y2="50.8" width="0.1524" layer="91"/>
+</segment>
+</net>
 </nets>
 </sheet>
