File: task/task-v/kicad/task-33/ground_truth/answer.kicad_sch (KiCad schematic)
At the start: 1 part, among them J1 Conn_02x20_Odd_Even

Commit message: Refine engineering task metadata and instructions
Parts:
- removed J1: Conn_02x20_Odd_Even, Connector_PinHeader_2.54mm:PinHeader_2x20_P2.54mm_Vertical, symbol Connector_Generic:Conn_02x20_Odd_Even
- added U1: nRF52840-QIAA, Package_DFN_QFN:Nordic_AQFN-73_7x7mm_P0.65mm, symbol nRF52840
Other:
- title: ASN02 HAT+ pinout correction -> ASN03 nRF52840 pinmux correction
