File: task/task-v/kicad/task-48/init_file/board.kicad_pcb (KiCad board)
At the start: 2 copper layers, 150 x 100 mm, 4 parts

Commit message: Refine engineering task metadata and instructions
Parts:
- removed the ? at (20.0, 20.0)
- removed the ? at (50.0, 1.50)
- removed the ? at (148.0, 50.0)
- removed the ? at (80.0, 60.0)
- added ?: , MountingHole:MountingHole_2.75mm_M2.5, F.Cu at (10.0, 15.0)
- added ?: , MountingHole:MountingHole_2.75mm_M2.5, F.Cu at (90.0, 25.0)
- added ?: , MountingHole:MountingHole_2.75mm_M2.5, F.Cu at (10.0, 75.0)
- added ?: , MountingHole:MountingHole_2.75mm_M2.5, F.Cu at (90.0, 80.0)
Other:
- board size 150 x 100 mm -> 100 x 100 mm
Changed lines of the file:
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@@
   )
   (net 0 "")
-  (net 1 "VCC")
-  (net 2 "GND")
-  ; Initial board: 150x100mm (too big for Hammond 1455C1201: slot 119x78mm)
-  (gr_rect (start 0 0) (end 150 100) (layer "Edge.Cuts") (width 0.1))
-  ; Some components, some too close to edges
-  (footprint "Package_SO:SOIC-8_3.9x4.9mm_P1.27mm" (layer "F.Cu") (at 20 20)
-    (reference "U1") (value "OPAMP")
-    (pad "1" smd rect (at -1.2 -1.27) (size 1.55 0.6)
-      (layers "F.Cu" "F.Paste" "F.Mask") (net 1 "VCC"))
+  (net 1 "GND")
+  (net 2 "VCC")
+  ; 4 non-plated mounting holes (np_thru_hole)
+  ; H1 at (10,15): Y=15 < analog_midline=50 — lowest Y, stays isolated (analog side)
+  (footprint "MountingHole:MountingHole_2.75mm_M2.5" (layer "F.Cu") (at 10 15)
+    (reference "H1") (value "MountingHole")
+    (attr through_hole)
+    (pad "" np_thru_hole circle (at 0 0) (size 2.5 2.5) (drill 2.5)
+      (layers "F.Cu" "B.Cu" "F.Mask" "B.Mask"))
   )
-  ; This component is within 3mm of edge y=0 — needs repositioning
-  (footprint "Resistor_SMD:R_0603_1608Metric" (layer "F.Cu") (at 50 1.5)
-    (reference "R1") (value "4.7k")
-    (pad "1" smd rect (at -0.8 0) (size 1.0 0.8)
-      (layers "F.Cu" "F.Paste" "F.Mask") (net 1 "VCC"))
+  ; H2 at (90,25): Y=25 < 50 but higher Y than H1 — will become plated GND
+  (footprint "MountingHole:MountingHole_2.75mm_M2.5" (layer "F.Cu") (at 90 25)
+    (reference "H2") (value "MountingHole")
+    (attr through_hole)
+    (pad "" np_thru_hole circle (at 0 0) (size 2.5 2.5) (drill 2.5)
+      (layers "F.Cu" "B.Cu" "F.Mask" "B.Mask"))
   )
-  ; This component is within 3mm of edge x=150 — needs repositioning
-  (footprint "Package_SO:SOIC-8_3.9x4.9mm_P1.27mm" (layer "F.Cu") (at 148 50)
-    (reference "U2") (value "ADC")
-    (pad "1" smd rect (at -1.2 -1.27) (size 1.55 0.6)
-      (layers "F.Cu" "F.Paste" "F.Mask") (net 2 "GND"))
+  ; H3 at (10,75): Y=75 > 50 — will become plated GND
+  (footprint "MountingHole:MountingHole_2.75mm_M2.5" (layer "F.Cu") (at 10 75)
+    (reference "H3") (value "MountingHole")
+    (attr through_hole)
+    (pad "" np_thru_hole circle (at 0 0) (size 2.5 2.5) (drill 2.5)
+      (layers "F.Cu" "B.Cu" "F.Mask" "B.Mask"))
   )
-  (footprint "Resistor_SMD:R_0603_1608Metric" (layer "F.Cu") (at 80 60)
-    (reference "R2") (value "10k")
-    (pad "1" smd rect (at -0.8 0) (size 1.0 0.8)
-      (layers "F.Cu" "F.Paste" "F.Mask") (net 2 "GND"))
+  ; H4 at (90,80): Y=80 > 50 — will become plated GND
+  (footprint "MountingHole:MountingHole_2.75mm_M2.5" (layer "F.Cu") (at 90 80)
+    (reference "H4") (value "MountingHole")
+    (attr through_hole)
+    (pad "" np_thru_hole circle (at 0 0) (size 2.5 2.5) (drill 2.5)
+      (layers "F.Cu" "B.Cu" "F.Mask" "B.Mask"))
   )
+  (gr_rect (start 0 0) (end 100 100) (layer "Edge.Cuts") (width 0.1))
 )
