File: task/task-v/kicad/task-12/ground_truth/answer.kicad_pcb (KiCad board)
At the start: 3 copper layers, 150 x 120 mm, 4 parts, among them U1 STM32F103, Y1 8MHz

Commit message: Fix GUI task startup configs
Other:
- copper layers 3 -> 4
Changed lines of the file:
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@@
     (0 "F.Cu" signal)
     (1 "In1.Cu" power)
+    (2 "In2.Cu" power)
     (31 "B.Cu" signal)
-    (36 "B.Paste" user)
-    (37 "F.Paste" user)
-    (38 "B.SilkS" user "B.Silkscreen")
-    (39 "F.SilkS" user "F.Silkscreen")
-    (40 "B.Mask" user)
-    (41 "F.Mask" user)
+    (34 "B.Paste" user)
+    (35 "F.Paste" user)
+    (36 "B.SilkS" user "B.Silkscreen")
+    (37 "F.SilkS" user "F.Silkscreen")
+    (38 "B.Mask" user)
+    (39 "F.Mask" user)
     (44 "Edge.Cuts" user)
   )
