File: task/task-v/kicad/task-19/init_file/board.kicad_pcb (KiCad board)
At the start: 2 copper layers, 100 x 80 mm, 5 parts

Commit message: Fix GUI task startup configs
Parts:
- removed ? (x4): , Package_SO:SOIC-8_3.9x4.9mm_P1.27mm
- removed ?: , Resistor_SMD:R_0603_1608Metric
- added R_TERM: 22R, Resistor_SMD:R_0603_1608Metric, F.Cu at (80.0, 30.0)
- added U1: 74HC04, Package_SO:SOIC-8_3.9x4.9mm_P1.27mm, F.Cu at (10.0, 30.0)
- added U2: 74HCT74, Package_SO:SOIC-8_3.9x4.9mm_P1.27mm, F.Cu at (50.0, 15.0)
- added U3: 74HCT74, Package_SO:SOIC-8_3.9x4.9mm_P1.27mm, F.Cu at (50.0, 30.0)
- added U4: 74HCT74, Package_SO:SOIC-8_3.9x4.9mm_P1.27mm, F.Cu at (50.0, 45.0)
Changed lines of the file:
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@@
   (net 2 "GND")
   (net 3 "VCC")
-  ; Source IC: U1 at (10, 30) — output pad drives CLK
   (footprint "Package_SO:SOIC-8_3.9x4.9mm_P1.27mm" (layer "F.Cu") (at 10 30)
-    (reference "U1") (value "74HC04")
+    (fp_text reference "U1" (at 0 -2) (layer "F.SilkS")
+      (effects (font (size 1 1) (thickness 0.15)))
+    )
+    (fp_text value "74HC04" (at 0 2) (layer "F.Fab")
+      (effects (font (size 1 1) (thickness 0.15)))
+    )
     (pad "3" thru_hole circle (at 0 0) (size 1.4 1.4) (drill 0.8)
       (layers "F.Cu" "B.Cu" "F.Mask" "B.Mask") (net 1 "CLK"))
   )
-  ; Load 1: U2 at (50, 15)
   (footprint "Package_SO:SOIC-8_3.9x4.9mm_P1.27mm" (layer "F.Cu") (at 50 15)
-    (reference "U2") (value "74HCT74")
+    (fp_text reference "U2" (at 0 -2) (layer "F.SilkS")
+      (effects (font (size 1 1) (thickness 0.15)))
+    )
+    (fp_text value "74HCT74" (at 0 2) (layer "F.Fab")
+      (effects (font (size 1 1) (thickness 0.15)))
+    )
     (pad "1" thru_hole circle (at 0 0) (size 1.4 1.4) (drill 0.8)
       (layers "F.Cu" "B.Cu" "F.Mask" "B.Mask") (net 1 "CLK"))
   )
-  ; Load 2: U3 at (50, 30)
   (footprint "Package_SO:SOIC-8_3.9x4.9mm_P1.27mm" (layer "F.Cu") (at 50 30)
-    (reference "U3") (value "74HCT74")
+    (fp_text reference "U3" (at 0 -2) (layer "F.SilkS")
+      (effects (font (size 1 1) (thickness 0.15)))
+    )
+    (fp_text value "74HCT74" (at 0 2) (layer "F.Fab")
+      (effects (font (size 1 1) (thickness 0.15)))
+    )
     (pad "1" thru_hole circle (at 0 0) (size 1.4 1.4) (drill 0.8)
       (layers "F.Cu" "B.Cu" "F.Mask" "B.Mask") (net 1 "CLK"))
   )
-  ; Load 3: U4 at (50, 45)
   (footprint "Package_SO:SOIC-8_3.9x4.9mm_P1.27mm" (layer "F.Cu") (at 50 45)
-    (reference "U4") (value "74HCT74")
+    (fp_text reference "U4" (at 0 -2) (layer "F.SilkS")
+      (effects (font (size 1 1) (thickness 0.15)))
+    )
+    (fp_text value "74HCT74" (at 0 2) (layer "F.Fab")
+      (effects (font (size 1 1) (thickness 0.15)))
+    )
     (pad "1" thru_hole circle (at 0 0) (size 1.4 1.4) (drill 0.8)
       (layers "F.Cu" "B.Cu" "F.Mask" "B.Mask") (net 1 "CLK"))
   )
-  ; Series termination resistor placeholder (scratch area, not connected)
   (footprint "Resistor_SMD:R_0603_1608Metric" (layer "F.Cu") (at 80 30)
-    (reference "R_TERM") (value "22R")
+    (fp_text reference "R_TERM" (at 0 -2) (layer "F.SilkS")
+      (effects (font (size 1 1) (thickness 0.15)))
+    )
+    (fp_text value "22R" (at 0 2) (layer "F.Fab")
+      (effects (font (size 1 1) (thickness 0.15)))
+    )
     (pad "1" smd rect (at -0.8 0) (size 1.0 0.8)
       (layers "F.Cu" "F.Paste" "F.Mask") (net 0 ""))
@@
       (layers "F.Cu" "F.Paste" "F.Mask") (net 0 ""))
   )
-  ; Star topology tracks: source (10,30) -> hub (30,30)
   (segment (start 10 30) (end 30 30) (width 0.2) (layer "F.Cu") (net 1))
-  ; Hub (30,30) -> U2 (50,15)
   (segment (start 30 30) (end 30 15) (width 0.2) (layer "F.Cu") (net 1))
   (segment (start 30 15) (end 50 15) (width 0.2) (layer "F.Cu") (net 1))
-  ; Hub (30,30) -> U3 (50,30)
   (segment (start 30 30) (end 50 30) (width 0.2) (layer "F.Cu") (net 1))
-  ; Hub (30,30) -> U4 (50,45)
   (segment (start 30 30) (end 30 45) (width 0.2) (layer "F.Cu") (net 1))
   (segment (start 30 45) (end 50 45) (width 0.2) (layer "F.Cu") (net 1))
