File: task/task-v/kicad/task-20/ground_truth/answer.kicad_pcb (KiCad board)
At the start: 2 copper layers, 80 x 80 mm, 8 parts

Commit message: Fix GUI task startup configs
Parts:
- removed ? (x2): , Connector_USB:USB_A_Molex_67643_Vertical
- removed ? (x2): , Connector_PinHeader_2.54mm:PinHeader_1x04_P2.54mm_Vertical
- removed ? (x4): , Package_TO_SOT_SMD:SOT-363_SC-70-6
- added D1: PRTR5V0U2X, Package_TO_SOT_SMD:SOT-363_SC-70-6, F.Cu at (8.00, 15.0)
- added D2: PRTR5V0U2X, Package_TO_SOT_SMD:SOT-363_SC-70-6, F.Cu at (8.00, 30.0)
- added D3: PRTR5V0U2X, Package_TO_SOT_SMD:SOT-363_SC-70-6, F.Cu at (8.00, 45.0)
- added D4: PRTR5V0U2X, Package_TO_SOT_SMD:SOT-363_SC-70-6, F.Cu at (8.00, 60.0)
- added J1: USB-A, Connector_USB:USB_A_Molex_67643_Vertical, F.Cu at (5.00, 15.0)
- added J2: USB-A, Connector_USB:USB_A_Molex_67643_Vertical, F.Cu at (5.00, 30.0)
- added J3: CONN-4P, Connector_PinHeader_2.54mm:PinHeader_1x04_P2.54mm_Vertical, F.Cu at (5.00, 45.0)
- added J4: CONN-4P, Connector_PinHeader_2.54mm:PinHeader_1x04_P2.54mm_Vertical, F.Cu at (5.00, 60.0)
Changed lines of the file:
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@@
   (net 4 "SIG_RX")
   (net 5 "GND")
-  ; Connectors unchanged
   (footprint "Connector_USB:USB_A_Molex_67643_Vertical" (layer "F.Cu") (at 5 15)
-    (reference "J1") (value "USB-A")
+    (fp_text reference "J1" (at 0 -2) (layer "F.SilkS")
+      (effects (font (size 1 1) (thickness 0.15)))
+    )
+    (fp_text value "USB-A" (at 0 2) (layer "F.Fab")
+      (effects (font (size 1 1) (thickness 0.15)))
+    )
     (pad "1" thru_hole circle (at 0 0) (size 1.5 1.5) (drill 0.8)
       (layers "F.Cu" "B.Cu" "F.Mask" "B.Mask") (net 1 "USB_DP"))
   )
   (footprint "Connector_USB:USB_A_Molex_67643_Vertical" (layer "F.Cu") (at 5 30)
-    (reference "J2") (value "USB-A")
+    (fp_text reference "J2" (at 0 -2) (layer "F.SilkS")
+      (effects (font (size 1 1) (thickness 0.15)))
+    )
+    (fp_text value "USB-A" (at 0 2) (layer "F.Fab")
+      (effects (font (size 1 1) (thickness 0.15)))
+    )
     (pad "1" thru_hole circle (at 0 0) (size 1.5 1.5) (drill 0.8)
       (layers "F.Cu" "B.Cu" "F.Mask" "B.Mask") (net 2 "USB_DM"))
   )
   (footprint "Connector_PinHeader_2.54mm:PinHeader_1x04_P2.54mm_Vertical" (layer "F.Cu") (at 5 45)
-    (reference "J3") (value "CONN-4P")
+    (fp_text reference "J3" (at 0 -2) (layer "F.SilkS")
+      (effects (font (size 1 1) (thickness 0.15)))
+    )
+    (fp_text value "CONN-4P" (at 0 2) (layer "F.Fab")
+      (effects (font (size 1 1) (thickness 0.15)))
+    )
     (pad "1" thru_hole circle (at 0 0) (size 1.7 1.7) (drill 1.0)
       (layers "F.Cu" "B.Cu" "F.Mask" "B.Mask") (net 3 "SIG_TX"))
   )
   (footprint "Connector_PinHeader_2.54mm:PinHeader_1x04_P2.54mm_Vertical" (layer "F.Cu") (at 5 60)
-    (reference "J4") (value "CONN-4P")
+    (fp_text reference "J4" (at 0 -2) (layer "F.SilkS")
+      (effects (font (size 1 1) (thickness 0.15)))
+    )
+    (fp_text value "CONN-4P" (at 0 2) (layer "F.Fab")
+      (effects (font (size 1 1) (thickness 0.15)))
+    )
     (pad "1" thru_hole circle (at 0 0) (size 1.7 1.7) (drill 1.0)
       (layers "F.Cu" "B.Cu" "F.Mask" "B.Mask") (net 4 "SIG_RX"))
   )
-  ; ESD arrays moved close to connectors (within 5mm of connector pads)
-  ; D1 moved to (8, 15): D1.pad1 at (8-1.2, 15)=(6.8,15), J1.pad at (5,15), dist=1.8mm <= 5mm
   (footprint "Package_TO_SOT_SMD:SOT-363_SC-70-6" (layer "F.Cu") (at 8 15)
-    (reference "D1") (value "PRTR5V0U2X")
+    (fp_text reference "D1" (at 0 -2) (layer "F.SilkS")
+      (effects (font (size 1 1) (thickness 0.15)))
+    )
+    (fp_text value "PRTR5V0U2X" (at 0 2) (layer "F.Fab")
+      (effects (font (size 1 1) (thickness 0.15)))
+    )
     (pad "1" smd rect (at -1.2 0) (size 0.7 0.5)
       (layers "F.Cu" "F.Paste" "F.Mask") (net 1 "USB_DP"))
@@
       (layers "F.Cu" "F.Paste" "F.Mask") (net 5 "GND"))
   )
-  ; D2 moved to (8, 30): D2.pad1 at (6.8,30), J2.pad at (5,30), dist=1.8mm <= 5mm
   (footprint "Package_TO_SOT_SMD:SOT-363_SC-70-6" (layer "F.Cu") (at 8 30)
-    (reference "D2") (value "PRTR5V0U2X")
+    (fp_text reference "D2" (at 0 -2) (layer "F.SilkS")
+      (effects (font (size 1 1) (thickness 0.15)))
+    )
+    (fp_text value "PRTR5V0U2X" (at 0 2) (layer "F.Fab")
+      (effects (font (size 1 1) (thickness 0.15)))
+    )
     (pad "1" smd rect (at -1.2 0) (size 0.7 0.5)
       (layers "F.Cu" "F.Paste" "F.Mask") (net 2 "USB_DM"))
@@
       (layers "F.Cu" "F.Paste" "F.Mask") (net 5 "GND"))
   )
-  ; D3 moved to (8, 45): D3.pad1 at (6.8,45), J3.pad at (5,45), dist=1.8mm <= 5mm
   (footprint "Package_TO_SOT_SMD:SOT-363_SC-70-6" (layer "F.Cu") (at 8 45)
-    (reference "D3") (value "PRTR5V0U2X")
+    (fp_text reference "D3" (at 0 -2) (layer "F.SilkS")
+      (effects (font (size 1 1) (thickness 0.15)))
+    )
+    (fp_text value "PRTR5V0U2X" (at 0 2) (layer "F.Fab")
+      (effects (font (size 1 1) (thickness 0.15)))
+    )
     (pad "1" smd rect (at -1.2 0) (size 0.7 0.5)
       (layers "F.Cu" "F.Paste" "F.Mask") (net 3 "SIG_TX"))
@@
       (layers "F.Cu" "F.Paste" "F.Mask") (net 5 "GND"))
   )
-  ; D4 moved to (8, 60): D4.pad1 at (6.8,60), J4.pad at (5,60), dist=1.8mm <= 5mm
   (footprint "Package_TO_SOT_SMD:SOT-363_SC-70-6" (layer "F.Cu") (at 8 60)
-    (reference "D4") (value "PRTR5V0U2X")
+    (fp_text reference "D4" (at 0 -2) (layer "F.SilkS")
+      (effects (font (size 1 1) (thickness 0.15)))
+    )
+    (fp_text value "PRTR5V0U2X" (at 0 2) (layer "F.Fab")
+      (effects (font (size 1 1) (thickness 0.15)))
+    )
     (pad "1" smd rect (at -1.2 0) (size 0.7 0.5)
       (layers "F.Cu" "F.Paste" "F.Mask") (net 4 "SIG_RX"))
