File: task/task-v/kicad/task-21/init_file/board.kicad_pcb (KiCad board)
At the start: 2 copper layers, 85 x 56 mm, 1 part

Commit message: Fix GUI task startup configs
Parts:
- removed ?: , Connector_PinHeader_2.54mm:PinHeader_2x20_P2.54mm_Vertical
- added J1: GPIO_HEADER, Connector_PinHeader_2.54mm:PinHeader_2x20_P2.54mm_Vertical, F.Cu at (30.0, 10.0)
Changed lines of the file:
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@@
   (net 1 "VCC")
   (net 2 "GND")
-  ; Initial board: 85x56mm rectangle, no mounting holes, no rounded corners
   (gr_rect (start 0 0) (end 85 56) (layer "Edge.Cuts") (width 0.1))
-  ; 2x20 GPIO header at (30, 10) -- needs to be repositioned
   (footprint "Connector_PinHeader_2.54mm:PinHeader_2x20_P2.54mm_Vertical" (layer "F.Cu") (at 30 10)
-    (reference "J1") (value "GPIO_HEADER")
+    (fp_text reference "J1" (at 0 -2) (layer "F.SilkS")
+      (effects (font (size 1 1) (thickness 0.15)))
+    )
+    (fp_text value "GPIO_HEADER" (at 0 2) (layer "F.Fab")
+      (effects (font (size 1 1) (thickness 0.15)))
+    )
     (pad "1" thru_hole circle (at 0 0) (size 1.7 1.7) (drill 1.0)
       (layers "F.Cu" "B.Cu" "F.Mask" "B.Mask") (net 1 "VCC"))
