File: task/task-v/kicad/task-22/init_file/board.kicad_pcb (KiCad board)
At the start: 2 copper layers, 150 x 100 mm, 4 parts

Commit message: Fix GUI task startup configs
Parts:
- removed ? (x2): , Package_SO:SOIC-8_3.9x4.9mm_P1.27mm
- removed ? (x2): , Resistor_SMD:R_0603_1608Metric
- added R1: 4.7k, Resistor_SMD:R_0603_1608Metric, F.Cu at (50.0, 1.50)
- added R2: 10k, Resistor_SMD:R_0603_1608Metric, F.Cu at (80.0, 60.0)
- added U1: OPAMP, Package_SO:SOIC-8_3.9x4.9mm_P1.27mm, F.Cu at (20.0, 20.0)
- added U2: ADC, Package_SO:SOIC-8_3.9x4.9mm_P1.27mm, F.Cu at (148.0, 50.0)
Changed lines of the file:
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@@
   (net 1 "VCC")
   (net 2 "GND")
-  ; Initial board: 150x100mm (too big for Hammond 1455C1201: slot 119x78mm)
   (gr_rect (start 0 0) (end 150 100) (layer "Edge.Cuts") (width 0.1))
-  ; Some components, some too close to edges
   (footprint "Package_SO:SOIC-8_3.9x4.9mm_P1.27mm" (layer "F.Cu") (at 20 20)
-    (reference "U1") (value "OPAMP")
+    (fp_text reference "U1" (at 0 -2) (layer "F.SilkS")
+      (effects (font (size 1 1) (thickness 0.15)))
+    )
+    (fp_text value "OPAMP" (at 0 2) (layer "F.Fab")
+      (effects (font (size 1 1) (thickness 0.15)))
+    )
     (pad "1" smd rect (at -1.2 -1.27) (size 1.55 0.6)
       (layers "F.Cu" "F.Paste" "F.Mask") (net 1 "VCC"))
   )
-  ; This component is within 3mm of edge y=0 — needs repositioning
   (footprint "Resistor_SMD:R_0603_1608Metric" (layer "F.Cu") (at 50 1.5)
-    (reference "R1") (value "4.7k")
+    (fp_text reference "R1" (at 0 -2) (layer "F.SilkS")
+      (effects (font (size 1 1) (thickness 0.15)))
+    )
+    (fp_text value "4.7k" (at 0 2) (layer "F.Fab")
+      (effects (font (size 1 1) (thickness 0.15)))
+    )
     (pad "1" smd rect (at -0.8 0) (size 1.0 0.8)
       (layers "F.Cu" "F.Paste" "F.Mask") (net 1 "VCC"))
   )
-  ; This component is within 3mm of edge x=150 — needs repositioning
   (footprint "Package_SO:SOIC-8_3.9x4.9mm_P1.27mm" (layer "F.Cu") (at 148 50)
-    (reference "U2") (value "ADC")
+    (fp_text reference "U2" (at 0 -2) (layer "F.SilkS")
+      (effects (font (size 1 1) (thickness 0.15)))
+    )
+    (fp_text value "ADC" (at 0 2) (layer "F.Fab")
+      (effects (font (size 1 1) (thickness 0.15)))
+    )
     (pad "1" smd rect (at -1.2 -1.27) (size 1.55 0.6)
       (layers "F.Cu" "F.Paste" "F.Mask") (net 2 "GND"))
   )
   (footprint "Resistor_SMD:R_0603_1608Metric" (layer "F.Cu") (at 80 60)
-    (reference "R2") (value "10k")
+    (fp_text reference "R2" (at 0 -2) (layer "F.SilkS")
+      (effects (font (size 1 1) (thickness 0.15)))
+    )
+    (fp_text value "10k" (at 0 2) (layer "F.Fab")
+      (effects (font (size 1 1) (thickness 0.15)))
+    )
     (pad "1" smd rect (at -0.8 0) (size 1.0 0.8)
       (layers "F.Cu" "F.Paste" "F.Mask") (net 2 "GND"))
