File: task/task-v/eagle/task-16/ground_truth/answer.sch (EAGLE design)
At the start: 0 parts

Commit message: Fix tasks identified in MoreOthers review
Parts:
- added C1: 100n, rcl:C
- added C2: 10u, rcl:C
- added LED1: red, led:LED
- added R1: 10k, rcl:R
- added R2: 47k, rcl:R
- added U1: 555, linear:555
Connections:
- new net CTRL: U1.CV
- new net DISCH: R1.2, R2.1, U1.DIS
- new net GND: C1.2, C2.2, LED1.C, U1.GND
- new net OUT: LED1.A, U1.Q
- new net TRIG_THRES: C1.1, R2.2, U1.THR, U1.TR
- new net VCC: C2.1, R1.1, U1.R, U1.V+
Changed lines of the file:
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@@
                 <wire x1="10" y1="10" x2="65" y2="10" width="0.1524" layer="91" />
                 <label x="12" y="10" size="1.778" layer="95" />
-                <pinref part="U1" gate="G$1" pin="VCC" />
+                <pinref part="U1" gate="G$1" pin="V+" />
+                <pinref part="U1" gate="G$1" pin="R" />
                 <pinref part="R1" gate="G$1" pin="1" />
                 <pinref part="C2" gate="G$1" pin="1" />
@@
                 <pinref part="C1" gate="G$1" pin="2" />
                 <pinref part="C2" gate="G$1" pin="2" />
-                <pinref part="LED1" gate="G$1" pin="K" />
+                <pinref part="LED1" gate="G$1" pin="C" />
               </segment>
             </net>
@@
                 <wire x1="10" y1="26" x2="65" y2="26" width="0.1524" layer="91" />
                 <label x="12" y="26" size="1.778" layer="95" />
-                <pinref part="U1" gate="G$1" pin="TRIG" />
-                <pinref part="U1" gate="G$1" pin="THRES" />
+                <pinref part="U1" gate="G$1" pin="TR" />
+                <pinref part="U1" gate="G$1" pin="THR" />
                 <pinref part="C1" gate="G$1" pin="1" />
                 <pinref part="R2" gate="G$1" pin="2" />
@@
                 <wire x1="10" y1="34" x2="65" y2="34" width="0.1524" layer="91" />
                 <label x="12" y="34" size="1.778" layer="95" />
-                <pinref part="U1" gate="G$1" pin="DISCH" />
+                <pinref part="U1" gate="G$1" pin="DIS" />
                 <pinref part="R1" gate="G$1" pin="2" />
                 <pinref part="R2" gate="G$1" pin="1" />
@@
                 <wire x1="10" y1="42" x2="65" y2="42" width="0.1524" layer="91" />
                 <label x="12" y="42" size="1.778" layer="95" />
-                <pinref part="U1" gate="G$1" pin="OUT" />
+                <pinref part="U1" gate="G$1" pin="Q" />
                 <pinref part="LED1" gate="G$1" pin="A" />
               </segment>
@@
                 <wire x1="10" y1="50" x2="65" y2="50" width="0.1524" layer="91" />
                 <label x="12" y="50" size="1.778" layer="95" />
-                <pinref part="U1" gate="G$1" pin="CTRL" />
+                <pinref part="U1" gate="G$1" pin="CV" />
               </segment>
             </net>
