File: task/task-c/eagle/task-22/ground_truth/answer.sch (EAGLE design)
At the start: 0 parts

Commit message: Sync harder Blender Eagle KiCad tasks to final
Parts:
- added C1, C2: 10u, polcap:E2,5-6
- added C3, C4: 10n, rcl:C-EU025-025X050
- added C5, C6: 27p, capacitor-wima:C2.5/2
- added D1: 1N4148, diode:1N4148
- added IC1: 16F84, microchip:PIC16F84AP
- added J1: (no value), PINHEAD:PINHD-1X20
- added Q1: (no value), special:XTAL/S
- added R1: 2.2k, rcl:R-EU_0207/10
- added U1: 78L05, linear:78LXXZ
Connections:
- new net +12V: C1.+, C3.2, J1.2, U1.VI
- new net A0: IC1.RA0, J1.4
- new net A1: IC1.RA1, J1.5
- new net A2: IC1.RA2, J1.6
- new net A3: IC1.RA3, J1.7
- new net A4: IC1.T0CKI/RA4, J1.8
- new net B0: IC1.RB0, J1.9
- new net B1: IC1.RB1, J1.10
- new net B2: IC1.RB2, J1.11
- new net B3: IC1.RB3, J1.12
- new net B4: IC1.RB4, J1.13
- new net B5: IC1.RB5, J1.14
- new net B6: IC1.RB6, J1.15, J1.18
- new net B7: IC1.RB7, J1.16, J1.17
- new net GND: C1.-, C2.-, C3.1, C4.1, C5.1, C6.1, IC1.VSS, J1.1, J1.20, U1.GND
- new net N$1: D1.C, IC1.!MCLR, J1.19
- new net N$2: D1.A, R1.1
- new net N$3: C5.2, IC1.OSC1, Q1.2
- new net N$4: C6.2, IC1.OSC2, Q1.1
- new net VCC: C2.+, C4.2, IC1.VDD, J1.3, R1.2, U1.VO
Other:
- note added: "1.0"
- note added: "PICSTAMP"
