File: task/task-v/kicad/task-11/init_file/design.kicad_pcb (KiCad board)
At the start: 2 copper layers, 140 x 110 mm, 8 parts, among them U1 ANT, U2 LNA, U3 BPF, U4 MIX, U5 AMP, U6 LPF, U7 ADC, U8 DAQ

Commit message: Sync harder Blender Eagle KiCad tasks to final
Connections:
- U1 pad 1: (no net) -> RF_IN
- U1 pad 2: (no net) -> RF_PREAMP
- U2 pad 1: (no net) -> RF_PREAMP
- U2 pad 2: (no net) -> RF_BANDPASS
- U3 pad 1: (no net) -> RF_BANDPASS
- U3 pad 2: (no net) -> RF_MIX
- U4 pad 1: (no net) -> RF_MIX
- U4 pad 2: (no net) -> RF_GAIN
- U5 pad 1: (no net) -> RF_GAIN
- U5 pad 2: (no net) -> RF_LOWPASS
- U6 pad 1: (no net) -> RF_LOWPASS
- U6 pad 2: (no net) -> RF_ADC
- U7 pad 1: (no net) -> RF_ADC
- U7 pad 2: (no net) -> RF_DATA
- U8 pad 1: (no net) -> RF_DATA
- U8 pad 2: (no net) -> RF_OUT
Changed lines of the file:
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@@
     (pad_to_mask_clearance 0)
   )
+  (net 0 "")
+  (net 1 "RF_IN")
+  (net 2 "RF_PREAMP")
+  (net 3 "RF_BANDPASS")
+  (net 4 "RF_MIX")
+  (net 5 "RF_GAIN")
+  (net 6 "RF_LOWPASS")
+  (net 7 "RF_ADC")
+  (net 8 "RF_DATA")
+  (net 9 "RF_OUT")
   (gr_rect (start 0 0) (end 140 110) (layer "Edge.Cuts") (width 0.05))
   (footprint "Connector_Coaxial:SMA_Amphenol_901-143-8RFX_Vertical"
@@
       (effects (font (size 1 1) (thickness 0.15)))
     )
-    (pad "1" smd rect (at -2 0 45) (size 1.5 0.8) (layers "F.Cu" "F.Paste" "F.Mask"))
-    (pad "2" smd rect (at 2 0 45) (size 1.5 0.8) (layers "F.Cu" "F.Paste" "F.Mask"))
+    (pad "1" smd rect (at -2 0 45) (size 1.5 0.8) (layers "F.Cu" "F.Paste" "F.Mask") (net 1 "RF_IN"))
+    (pad "2" smd rect (at 2 0 45) (size 1.5 0.8) (layers "F.Cu" "F.Paste" "F.Mask") (net 2 "RF_PREAMP"))
   )
   (footprint "Package_SO:SOIC-8_3.9x4.9mm_P1.27mm"
@@
       (effects (font (size 1 1) (thickness 0.15)))
     )
-    (pad "1" smd rect (at -2 0 135) (size 1.5 0.8) (layers "F.Cu" "F.Paste" "F.Mask"))
-    (pad "2" smd rect (at 2 0 135) (size 1.5 0.8) (layers "F.Cu" "F.Paste" "F.Mask"))
+    (pad "1" smd rect (at -2 0 135) (size 1.5 0.8) (layers "F.Cu" "F.Paste" "F.Mask") (net 2 "RF_PREAMP"))
+    (pad "2" smd rect (at 2 0 135) (size 1.5 0.8) (layers "F.Cu" "F.Paste" "F.Mask") (net 3 "RF_BANDPASS"))
   )
   (footprint "Package_SO:SOIC-8_3.9x4.9mm_P1.27mm"
@@
       (effects (font (size 1 1) (thickness 0.15)))
     )
-    (pad "1" smd rect (at -2 0 270) (size 1.5 0.8) (layers "F.Cu" "F.Paste" "F.Mask"))
-    (pad "2" smd rect (at 2 0 270) (size 1.5 0.8) (layers "F.Cu" "F.Paste" "F.Mask"))
+    (pad "1" smd rect (at -2 0 270) (size 1.5 0.8) (layers "F.Cu" "F.Paste" "F.Mask") (net 3 "RF_BANDPASS"))
+    (pad "2" smd rect (at 2 0 270) (size 1.5 0.8) (layers "F.Cu" "F.Paste" "F.Mask") (net 4 "RF_MIX"))
   )
   (footprint "Package_SO:SOIC-8_3.9x4.9mm_P1.27mm"
@@
       (effects (font (size 1 1) (thickness 0.15)))
     )
-    (pad "1" smd rect (at -2 0 0) (size 1.5 0.8) (layers "F.Cu" "F.Paste" "F.Mask"))
-    (pad "2" smd rect (at 2 0 0) (size 1.5 0.8) (layers "F.Cu" "F.Paste" "F.Mask"))
+    (pad "1" smd rect (at -2 0 0) (size 1.5 0.8) (layers "F.Cu" "F.Paste" "F.Mask") (net 4 "RF_MIX"))
+    (pad "2" smd rect (at 2 0 0) (size 1.5 0.8) (layers "F.Cu" "F.Paste" "F.Mask") (net 5 "RF_GAIN"))
   )
   (footprint "Package_SO:SOIC-8_3.9x4.9mm_P1.27mm"
@@
       (effects (font (size 1 1) (thickness 0.15)))
     )
-    (pad "1" smd rect (at -2 0 180) (size 1.5 0.8) (layers "F.Cu" "F.Paste" "F.Mask"))
-    (pad "2" smd rect (at 2 0 180) (size 1.5 0.8) (layers "F.Cu" "F.Paste" "F.Mask"))
+    (pad "1" smd rect (at -2 0 180) (size 1.5 0.8) (layers "F.Cu" "F.Paste" "F.Mask") (net 5 "RF_GAIN"))
+    (pad "2" smd rect (at 2 0 180) (size 1.5 0.8) (layers "F.Cu" "F.Paste" "F.Mask") (net 6 "RF_LOWPASS"))
   )
   (footprint "Package_SO:SOIC-8_3.9x4.9mm_P1.27mm"
@@
       (effects (font (size 1 1) (thickness 0.15)))
     )
-    (pad "1" smd rect (at -2 0 90) (size 1.5 0.8) (layers "F.Cu" "F.Paste" "F.Mask"))
-    (pad "2" smd rect (at 2 0 90) (size 1.5 0.8) (layers "F.Cu" "F.Paste" "F.Mask"))
+    (pad "1" smd rect (at -2 0 90) (size 1.5 0.8) (layers "F.Cu" "F.Paste" "F.Mask") (net 6 "RF_LOWPASS"))
+    (pad "2" smd rect (at 2 0 90) (size 1.5 0.8) (layers "F.Cu" "F.Paste" "F.Mask") (net 7 "RF_ADC"))
   )
   (footprint "Package_SO:SOIC-16_3.9x9.9mm_P1.27mm"
@@
       (effects (font (size 1 1) (thickness 0.15)))
     )
-    (pad "1" smd rect (at -2 0 45) (size 1.5 0.8) (layers "F.Cu" "F.Paste" "F.Mask"))
-    (pad "2" smd rect (at 2 0 45) (size 1.5 0.8) (layers "F.Cu" "F.Paste" "F.Mask"))
+    (pad "1" smd rect (at -2 0 45) (size 1.5 0.8) (layers "F.Cu" "F.Paste" "F.Mask") (net 7 "RF_ADC"))
+    (pad "2" smd rect (at 2 0 45) (size 1.5 0.8) (layers "F.Cu" "F.Paste" "F.Mask") (net 8 "RF_DATA"))
   )
   (footprint "Package_SO:SOIC-16_3.9x9.9mm_P1.27mm"
@@
       (effects (font (size 1 1) (thickness 0.15)))
     )
-    (pad "1" smd rect (at -2 0 315) (size 1.5 0.8) (layers "F.Cu" "F.Paste" "F.Mask"))
-    (pad "2" smd rect (at 2 0 315) (size 1.5 0.8) (layers "F.Cu" "F.Paste" "F.Mask"))
+    (pad "1" smd rect (at -2 0 315) (size 1.5 0.8) (layers "F.Cu" "F.Paste" "F.Mask") (net 8 "RF_DATA"))
+    (pad "2" smd rect (at 2 0 315) (size 1.5 0.8) (layers "F.Cu" "F.Paste" "F.Mask") (net 9 "RF_OUT"))
   )
 )
