File: task/quantified/cli-kicad-layout-optimization/task-01/init_file/seed_board.kicad_pcb (KiCad board)
At the start: 80 x 52 mm, 7 parts

Commit message: Repair KiCad 10.0.2 tasks and evaluators
Parts:
- C1: value (none) -> 100nF; footprint Engiworld:C1 -> (none)
- C2: value (none) -> 100nF; footprint Engiworld:C2 -> (none)
- C3: value (none) -> 1uF; footprint Engiworld:C3 -> (none)
- J1: value (none) -> INPUT; footprint Engiworld:J1 -> (none)
- J2: value (none) -> OUTPUT; footprint Engiworld:J2 -> (none)
- L1: value (none) -> 10uH; footprint Engiworld:L1 -> (none)
- U1: value (none) -> MIXED_SIGNAL_MCU; footprint Engiworld:U1 -> (none)
Routing:
- net C3_U1: track 27.2 -> 25.8 mm
- net C1_U1: track 29.2 -> 27.8 mm
- net C2_U1: track 27.8 -> 26.4 mm
- net STITCH: vias 8 -> 0
Other:
- copper layers 0 -> 2
