File: task/quantified/cli-kicad-layout-optimization/task-02/ground_truth/optimized_board.kicad_pcb (KiCad board)
At the start: 96 x 58 mm, 7 parts

Commit message: Repair KiCad 10.0.2 tasks and evaluators
Parts:
- C1: value (none) -> 100nF; footprint Engiworld:C1 -> (none)
- C2: value (none) -> 100nF; footprint Engiworld:C2 -> (none)
- J1: value (none) -> DIFF_CONNECTOR; footprint Engiworld:J1 -> (none)
- J2: value (none) -> BYPASS_CONNECTOR; footprint Engiworld:J2 -> (none)
- R1: value (none) -> 49.9R; footprint Engiworld:R1 -> (none)
- R2: value (none) -> 49.9R; footprint Engiworld:R2 -> (none)
- U1: value (none) -> DIFF_DRIVER; footprint Engiworld:U1 -> (none)
Routing:
- net U1_R2: track 26.7 -> 25.8 mm
- net U1_R1: track 26.7 -> 25.8 mm
- net R2_J1: track 34.5 -> 33.7 mm, vias 0 -> 1
- net R1_J1: track 34.5 -> 33.7 mm, vias 0 -> 1
- net J2_C1: track 34.4 -> 33.6 mm, vias 0 -> 1
- net J2_C2: track 23.3 -> 23.9 mm
- net STITCH: vias 3 -> 0
Other:
- copper layers 0 -> 2
