File: task/quantified/cli-kicad-layout-optimization/task-04/init_file/seed_board.kicad_pcb (KiCad board)
At the start: 88 x 70 mm, 8 parts

Commit message: Repair KiCad 10.0.2 tasks and evaluators
Parts:
- C1: value (none) -> C1; footprint Engiworld:C1 -> (none)
- J1: value (none) -> J1; footprint Engiworld:J1 -> (none)
- J2: value (none) -> J2; footprint Engiworld:J2 -> (none)
- TP1: value (none) -> POGO_TEST; footprint Engiworld:TP1 -> (none)
- TP2: value (none) -> POGO_TEST; footprint Engiworld:TP2 -> (none)
- TP3: value (none) -> POGO_TEST; footprint Engiworld:TP3 -> (none)
- TP4: value (none) -> POGO_TEST; footprint Engiworld:TP4 -> (none)
- U1: value (none) -> U1; footprint Engiworld:U1 -> (none)
Routing:
- net TP4_U1: track 30.5 -> 28.7 mm
- net TP1_U1: track 30.5 -> 28.7 mm
- net TP3_U1: track 28.6 -> 27.5 mm
- net TP2_U1: track 28.6 -> 27.5 mm
- net C1_U1: track 26.0 -> 25.0 mm
- net STITCH: vias 8 -> 0
Other:
- copper layers 0 -> 2
