File: task/quantified/cli-kicad-layout-optimization/task-05/init_file/seed_board.kicad_pcb (KiCad board)
At the start: 76 x 76 mm, 7 parts

Commit message: Repair KiCad 10.0.2 tasks and evaluators
Parts:
- A1: value (none) -> A1; footprint Engiworld:A1 -> (none)
- C1: value (none) -> C1; footprint Engiworld:C1 -> (none)
- C2: value (none) -> C2; footprint Engiworld:C2 -> (none)
- J1: value (none) -> J1; footprint Engiworld:J1 -> (none)
- L1: value (none) -> L1; footprint Engiworld:L1 -> (none)
- TP1: value (none) -> TP1; footprint Engiworld:TP1 -> (none)
- U1: value (none) -> U1; footprint Engiworld:U1 -> (none)
Routing:
- net L1_J1: track 4.47 -> 3.86 mm
- net A1_C1: track 25.1 -> 24.4 mm
- net STITCH: vias 8 -> 0
Other:
- copper layers 0 -> 2
