File: task/task-c/kicad/task-08/ground_truth/design.kicad_pcb (KiCad board)
At the start: 2 copper layers, 5 parts, among them Q1 BC547, U1 LM7805

Commit message: Repair KiCad 10.0.2 tasks and evaluators
Parts:
- C1: footprint Capacitor_SMD:C_0402_1005Metric -> Capacitors_SMD:C_0402
- D1: footprint LED_SMD:LED_0603_1608Metric -> LEDs:LED_0603
- Q1: footprint Package_TO_SOT_THT:TO-92_Inline -> TO_SOT_Packages_THT:TO-92_Inline
- R1: footprint Resistor_SMD:R_0603_1608Metric -> Resistors_SMD:R_0603
- U1: footprint Package_TO_SOT_THT:TO-220-3_Vertical -> TO_SOT_Packages_THT:TO-220_Vertical
