File: task/task-c/kicad/task-08/ground_truth/design.kicad_sch (KiCad schematic)
At the start: 5 parts, among them Q1 BC547, U1 LM7805

Commit message: Repair KiCad 10.0.2 tasks and evaluators
Parts:
- removed Q1: BC547, symbol Device:Q_NPN_BCE
- added Q1: BC547, symbol Transistor_BJT:Q_NPN_BCE
- U1: footprint Package_TO_SOT_THT:TO-220-3_Vertical -> (none)
Connections:
- net GND: now also C1.2, R1.2, U1.2 (GND), Q1.3 (E)
- net VCC: now also C1.1, R1.1, U1.1 (VI)
- net SIG_B: now reaches D1.1 (K)
- net SIG_B: now also Q1.2 (C)
- net SIG_A: now reaches D1.2 (A)
- net SIG_A: now also Q1.1 (B)
- net +5V: now reaches U1.3 (VO)
