File: task/task-v/kicad/task-02/ground_truth/buck.kicad_sch (KiCad schematic)
At the start: 24 parts, among them J1 VIN_CONN, Q1 FDMC86102, Q2 FDMC86102, U1 LM5116

Commit message: Repair KiCad 10.0.2 tasks and evaluators
Parts:
- removed J1: VIN_CONN, symbol Connector:Conn_01x02_Pin
- removed Q1, Q2: FDMC86102, symbol Device:Q_NMOS_GSD
- removed U1: LM5116, symbol Device:IC
- added J1: VIN_CONN, symbol Benchmark:Connector_02_Abstract
- added Q1, Q2: FDMC86102, symbol Benchmark:MOSFET_GSD_Abstract
- added U1: LM5116, symbol Benchmark:IC_06_Abstract
- C1, C10, C11, C12, C13, C2, C3, C4, C5, C6, C7, C8, C9, D1, L1, R1, R2, R3, R4, R_SENSE: ConnectivityScope (none) -> specified_by_source
Connections:
- net VBUCK: now also C1.1, C2.1, C3.1, C4.1, C5.1, C6.1, L1.2, R1.1
- new net BOOT: C13.2, D1.1 (K)
- new net COMP: C11.1, C12.1, R3.1
- new net EN: R4.2
- new net FB: R1.2, R2.1
- new net GND: C1.2, C10.2, C11.2, C12.2, C2.2, C3.2, C4.2, C5.2, C6.2, C7.2, C8.2, C9.2, R2.2, R3.2, R_SENSE.2
- new net SW: C13.1, L1.1, R_SENSE.1
- new net VIN: C10.1, C7.1, C8.1, C9.1, D1.2 (A), R4.1
- no-connect marks 0 -> 14
Other:
- company: SCH01 Benchmark -> EngiWorld
