File: task/task-v/kicad/task-02/ground_truth/ldo.kicad_sch (KiCad schematic)
At the start: 15 parts, among them U2 MIC5205-3.3YM5

Commit message: Repair KiCad 10.0.2 tasks and evaluators
Parts:
- removed D2: LED_GREEN, symbol Device:D
- removed U2: MIC5205-3.3YM5, symbol Device:IC
- added D2: LED_GREEN, symbol Device:LED
- added U2: MIC5205-3.3YM5, symbol Benchmark:IC_04_Abstract
- C14, C15, C16, C17, C18, C19, C20, C21, C22, C23, C24, R5, R6: ConnectivityScope (none) -> specified_by_source
Connections:
- net VBUCK: now also C14.1, C15.1, C16.1, C24.1
- net VLDO: now also C17.1, C18.1, C19.1, C20.1, C21.1, C22.1, C23.1, R5.1, D2.2 (A)
- new net GND: C14.2, C15.2, C16.2, C17.2, C18.2, C19.2, C20.2, C21.2, C22.2, C23.2, C24.2, R6.2
- new net LDO_EN: R5.2
- new net LED_A: D2.1 (K), R6.1
- no-connect marks 0 -> 4
Other:
- company: SCH01 Benchmark -> EngiWorld
- title: Power Supply - Ldo Section -> Power Supply - LDO Section
