File: task/task-v/kicad/task-03/init_file/mcu.kicad_sch (KiCad schematic)
At the start: 9 parts, among them U1 STM32F103C8T6, U2 IS62WV51216BLL

Commit message: Repair KiCad 10.0.2 tasks and evaluators
Parts:
- removed U1: STM32F103C8T6, Package_QFP:LQFP-48_7x7mm_P0.5mm, symbol Device:IC
- removed U2: IS62WV51216BLL, Package_SO:TSOP-II-44_10.16x18.41mm_P0.8mm, symbol Device:IC
- added U1: STM32F103C8T6, Package_QFP:LQFP-48_7x7mm_P0.5mm, symbol MCU_ST_STM32F1:STM32F103C8Tx
- added U2: IS62WV51216BLL, Package_SO:TSOP-II-44_10.16x18.41mm_P0.8mm, symbol EngiWorld:IS62WV51216BLL
- C1, C2, C3, C4: Net1 3V3 -> (none); Net2 GND -> (none)
- R1: Net1 3V3 -> (none); Net2 CE_N -> (none)
- R2: Net1 3V3 -> (none); Net2 OE_N -> (none)
- R3: Net1 3V3 -> (none); Net2 WE_N -> (none)
Connections:
- new net +3V3: C1.1, C2.1, C3.1, C4.1, R1.1, R2.1, R3.1, U1.1 (VBAT), U1.24 (VDD), U1.36 (VDD), U1.48 (VDD), U1.9 (VDDA), U2.11 (VDD), U2.33 (VDD)
- new net CE_N: R1.2, U2.6 (~{CS1})
- new net GND: C1.2, C2.2, C3.2, C4.2, U1.23 (VSS), U1.35 (VSS), U1.47 (VSS), U1.8 (VSSA), U2.12 (GND), U2.34 (GND)
- new net OE_N: R2.2, U2.41 (~{OE})
- new net WE_N: R3.2, U2.17 (~{WE})
- no-connect marks 0 -> 60
Other:
- company: SCH02 Benchmark -> EngiWorld
