File: task/multi/gui-4-librecad-freecad-kicad-blender/task-06/ground_truth/stage3_fan_control_panel_board.kicad_pcb (KiCad board)
At the start: 145 x 95 mm, 0 parts

Commit message: 更新修复后的正式 task 数据
Parts:
- added DS1: OLED display, , F.Cu at (72.5, 75.0)
- added J1: Fan header 4-pin, , F.Cu at (22.0, 18.0)
- added SW1: Rotary encoder, , F.Cu at (116.0, 47.5)
- added SW2: Button UP, , F.Cu at (43.0, 18.0)
- added SW3: Button DOWN, , F.Cu at (58.0, 18.0)
- added SW4: Button MODE, , F.Cu at (73.0, 18.0)
- added SW5: Button SET, , F.Cu at (88.0, 18.0)
Other:
- copper layers 0 -> 2
- board text added: "BTN-SET"
