File: task/multi/gui-4-librecad-freecad-kicad-blender/task-07/ground_truth/stage3_sbc_hat_mount_plate_board.kicad_pcb (KiCad board)
At the start: 85 x 65 mm, 0 parts

Commit message: 更新修复后的正式 task 数据
Parts:
- added J1: GPIO40 header 2x20, , F.Cu at (42.5, 50.0)
- added J2: I2C header 1x4, , F.Cu at (66.0, 15.0)
- added J3: Power input 2-pin, , F.Cu at (72.0, 32.0)
- added U1: EEPROM SOIC-8, , F.Cu at (22.0, 25.0)
Other:
- copper layers 0 -> 2
