File: task/multi/gui-4-librecad-freecad-kicad-blender/task-08/ground_truth/stage3_terminal_cover_long_board.kicad_pcb (KiCad board)
At the start: 165 x 52 mm, 0 parts

Commit message: 更新修复后的正式 task 数据
Parts:
- added PWR1: 24V GND power input, , F.Cu at (82.5, 45.0)
- added TERM1: 2-pin terminal channel 1, , F.Cu at (19.5, 26.0)
- added TERM2: 2-pin terminal channel 2, , F.Cu at (37.5, 26.0)
- added TERM3: 2-pin terminal channel 3, , F.Cu at (55.5, 26.0)
- added TERM4: 2-pin terminal channel 4, , F.Cu at (73.5, 26.0)
- added TERM5: 2-pin terminal channel 5, , F.Cu at (91.5, 26.0)
- added TERM6: 2-pin terminal channel 6, , F.Cu at (109.5, 26.0)
- added TERM7: 2-pin terminal channel 7, , F.Cu at (127.5, 26.0)
- added TERM8: 2-pin terminal channel 8, , F.Cu at (145.5, 26.0)
Other:
- copper layers 0 -> 2
- board text added: "FREECAD_TO_KICAD"
- board text added: "TERM1 TERM2 TERM3 TERM4"
- board text added: "TERM5 TERM6 TERM7 TERM8"
- board text removed: "TERM1"
- board text removed: "TERM2"
- board text removed: "TERM3"
- board text removed: "TERM4"
- board text removed: "TERM5"
- board text removed: "TERM6"
- board text removed: "TERM7"
- board text removed: "TERM8"
