File: task/multi/gui-4-librecad-freecad-kicad-blender/task-09/ground_truth/stage3_wearable_charger_cradle_board.kicad_pcb (KiCad board)
At the start: 105 x 48 mm, 0 parts

Commit message: 更新修复后的正式 task 数据
Parts:
- added CHG-U1: CHARGER_IC, Connector_PinHeader_2.54mm:PinHeader_1x02_P2.54mm_Vertical_SMD_Pin1Left, F.Cu at (47.0, 14.0)
- added MAGNET-M1: MAGNET_MARKER, Connector_PinHeader_2.54mm:PinHeader_1x02_P2.54mm_Vertical_SMD_Pin1Left, F.Cu at (72.0, 24.0)
- added NTC-R1: NTC_SENSOR, Connector_PinHeader_2.54mm:PinHeader_1x02_P2.54mm_Vertical_SMD_Pin1Left, F.Cu at (70.0, 14.0)
- added POGO-P1: POGO_POS_CONTACT, Connector_PinHeader_2.54mm:PinHeader_1x02_P2.54mm_Vertical_SMD_Pin1Left, F.Cu at (47.0, 24.0)
- added POGO-P2: POGO_NEG_CONTACT, Connector_PinHeader_2.54mm:PinHeader_1x02_P2.54mm_Vertical_SMD_Pin1Left, F.Cu at (56.0, 24.0)
- added USB-J1: USB_INPUT, Connector_PinHeader_2.54mm:PinHeader_1x02_P2.54mm_Vertical_SMD_Pin1Left, F.Cu at (30.0, 14.0)
Other:
- copper layers 0 -> 2
- board text added: "FREECAD_TO_KICAD"
